File: CONN.kicad_sch (KiCad schematic)
At the start: 24 parts, among them CN1 5019530507, CN2 5019530507, U1 SRV05-4, U2 SRV05-4

Commit message: All 0603 version
Parts:
- C1, C2, C3, C4: footprint Capacitor_SMD:C_0402_1005Metric -> Capacitor_SMD:C_0603_1608Metric
- D1, D2: footprint LED_SMD:LED_0402_1005Metric -> LED_SMD:LED_0603_1608Metric
- R2, R3, R4, R5: footprint Resistor_SMD:R_0402_1005Metric -> Resistor_SMD:R_0603_1608Metric
Changed lines of the file:
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@@
       (effects (font (size 1.27 1.27)))
     )
-    (property "Footprint" "LED_SMD:LED_0402_1005Metric" (at 230.124 51.943 0)
+    (property "Footprint" "LED_SMD:LED_0603_1608Metric" (at 230.124 51.943 0)
       (effects (font (size 1.27 1.27)) hide)
     )
@@
       (effects (font (size 1.27 1.27)))
     )
-    (property "Footprint" "Resistor_SMD:R_0402_1005Metric" (at 134.874 132.461 90)
+    (property "Footprint" "Resistor_SMD:R_0603_1608Metric" (at 134.874 132.461 90)
       (effects (font (size 1.27 1.27)) hide)
     )
@@
       (effects (font (size 1.27 1.27)))
     )
-    (property "Footprint" "LED_SMD:LED_0402_1005Metric" (at 230.124 41.783 0)
+    (property "Footprint" "LED_SMD:LED_0603_1608Metric" (at 230.124 41.783 0)
       (effects (font (size 1.27 1.27)) hide)
     )
@@
       (effects (font (size 1.27 1.27)))
     )
-    (property "Footprint" "Capacitor_SMD:C_0402_1005Metric" (at 67.564 137.3378 0)
+    (property "Footprint" "Capacitor_SMD:C_0603_1608Metric" (at 67.564 137.3378 0)
       (effects (font (size 1.27 1.27)) hide)
     )
@@
       (effects (font (size 1.27 1.27)))
     )
-    (property "Footprint" "Resistor_SMD:R_0402_1005Metric" (at 134.874 117.221 90)
+    (property "Footprint" "Resistor_SMD:R_0603_1608Metric" (at 134.874 117.221 90)
       (effects (font (size 1.27 1.27)) hide)
     )
@@
       (effects (font (size 1.27 1.27)))
     )
-    (property "Footprint" "Capacitor_SMD:C_0402_1005Metric" (at 67.564 122.0978 0)
+    (property "Footprint" "Capacitor_SMD:C_0603_1608Metric" (at 67.564 122.0978 0)
       (effects (font (size 1.27 1.27)) hide)
     )
@@
       (effects (font (size 1.27 1.27)))
     )
-    (property "Footprint" "Resistor_SMD:R_0402_1005Metric" (at 134.874 101.981 90)
+    (property "Footprint" "Resistor_SMD:R_0603_1608Metric" (at 134.874 101.981 90)
       (effects (font (size 1.27 1.27)) hide)
     )
@@
       (effects (font (size 1.27 1.27)))
     )
-    (property "Footprint" "Capacitor_SMD:C_0402_1005Metric" (at 67.564 106.8578 0)
+    (property "Footprint" "Capacitor_SMD:C_0603_1608Metric" (at 67.564 106.8578 0)
       (effects (font (size 1.27 1.27)) hide)
     )
@@
       (effects (font (size 1.27 1.27)))
     )
-    (property "Footprint" "Capacitor_SMD:C_0402_1005Metric" (at 67.564 91.6178 0)
+    (property "Footprint" "Capacitor_SMD:C_0603_1608Metric" (at 67.564 91.6178 0)
       (effects (font (size 1.27 1.27)) hide)
     )
@@
       (effects (font (size 1.27 1.27)))
     )
-    (property "Footprint" "Resistor_SMD:R_0402_1005Metric" (at 134.874 86.741 90)
-      (effects (font (size 1.27 1.27)) hide)
-    )
+    (property "Footprint" "Resistor_SMD:R_0603_1608Metric" (at 134.874 86.741 90)
+      (effects (font (size 1.27 1.27)) hide)
+    )

Commit message: Official version
Connections:
- net P0_MRXIN: now also L1.2; no longer L1.1
- net P0_MRXIP: now also L1.1; no longer L1.2
- net P0_MTXON: now also L1.6; no longer L1.5
- net P0_MTXOP: now also L1.5; no longer L1.6
- net P0_RXIN: now also L1.23; no longer L1.24
- net P0_RXIP: now also L1.24; no longer L1.23
- net P0_TXON: now also L1.19; no longer L1.20
- net P0_TXOP: now also L1.20; no longer L1.19
- net P1_MRXIN: now also L1.8; no longer L1.7
- net P1_MRXIP: now also L1.7; no longer L1.8
- net P1_MTXON: now also L1.12; no longer L1.11
- net P1_MTXOP: now also L1.11; no longer L1.12
- net P1_RXIN: now also L1.17; no longer L1.18
- net P1_RXIP: now also L1.18; no longer L1.17
- net P1_TXON: now also L1.13; no longer L1.14
- net P1_TXOP: now also L1.14; no longer L1.13
