File: EtherCAT_CONN.kicad_sch (KiCad schematic)
At the start: 4 parts, among them J2 Conn_01x12

Commit message: Official version
Parts:
- removed J2: Conn_01x12, Connector_PinHeader_1.27mm:ECAT, symbol Connector_Generic:Conn_01x12
- added H4: MountingHole, EXTRA IC:M1.6, symbol Mechanical:MountingHole
- added J1: Conn_01x20, Connector_PinHeader_1.27mm:ECAT_20pin, symbol Connector_Generic:Conn_01x20
- added J2: Conn_01x06, Connector_JST:JST_SH_BM06B-SRSS-TB_1x06-1MP_P1.00mm_Vertical, symbol Connector_Generic:Conn_01x06
- H1, H2, H3: footprint EXTRA IC:MountingHole_1.7mm_M1.6 -> EXTRA IC:M1.6
Connections:
- net A3V3: now also J1.10 (Pin_10)
- net CONN/P0_ACT: now also J1.20 (Pin_20)
- net CONN/P0_RXIN: now also J1.18 (Pin_18)
- net CONN/P0_RXIP: now also J1.17 (Pin_17)
- net CONN/P0_TXON: now also J1.16 (Pin_16)
- net CONN/P0_TXOP: now also J1.15 (Pin_15)
- net CONN/P1_ACT: now also J1.19 (Pin_19)
- net CONN/P1_RXIN: now also J1.14 (Pin_14)
- net CONN/P1_RXIP: now also J1.13 (Pin_13)
- net CONN/P1_TXON: now also J1.12 (Pin_12)
- net CONN/P1_TXOP: now also J1.11 (Pin_11)
- net GND: now also J1.1 (Pin_1), J1.9 (Pin_9), J2.5 (Pin_5)
- new net +5V: J1.2 (Pin_2), J2.6 (Pin_6)
- new net DEBUG0: J1.8 (Pin_8)
- new net DEBUG1: J1.7 (Pin_7)
- new net SWCLK: J1.3 (Pin_3), J2.1 (Pin_1)
- new net SWDIO: J1.4 (Pin_4), J2.2 (Pin_2)
- new net USART_RX: J1.5 (Pin_5), J2.3 (Pin_3)
- new net USART_TX: J1.6 (Pin_6), J2.4 (Pin_4)
